File: ll-irm-psu-board.kicad_sch (KiCad schematic)
At the start: 0 parts

Commit message: adding schematic
Parts:
- added D1: PWR LED, symbol Device:LED
- added J1: 230VAC, symbol Connector_Generic:Conn_01x02
- added J2: 5V+ Output, symbol Connector_Generic:Conn_01x02
- added PS1: IRM-03-5, Converter_ACDC:Converter_ACDC_MeanWell_IRM-03-xx_THT, symbol Converter_ACDC:IRM-03-5
- added R1: 2K, symbol Device:R
Connections:
- new net: J1.1 (Pin_1), PS1.3 (AC/N)
- new net: J1.2 (Pin_2), PS1.1 (AC/L)
- new net: D1.2 (A), J2.1 (Pin_1), PS1.16 (+Vo)
- new net: D1.1 (K), R1.1
- new net GND: J2.2 (Pin_2), PS1.14 (-Vo), R1.2
Changed lines of the file:
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@@
     (company "LL DIY")
+  )
+  (junction (at 81.788 62.992) (diameter 0) (color 0 0 0 0)
+  )
+  (junction (at 123.698 64.516) (diameter 0) (color 0 0 0 0)
+  )
+  (junction (at 118.618 59.436) (diameter 0) (color 0 0 0 0)
+  )
+  (junction (at 81.026 60.452) (diameter 0) (color 0 0 0 0)
+  )
+  (wire (pts (xy 145.034 45.974) (xy 145.034 48.768))
+    (stroke (width 0) (type default) (color 0 0 0 0))
+  )
+  (wire (pts (xy 81.026 60.452) (xy 94.234 60.452))
+    (stroke (width 0) (type default) (color 0 0 0 0))
+  )
+  (wire (pts (xy 128.016 45.974) (xy 132.842 45.974))
+    (stroke (width 0) (type default) (color 0 0 0 0))
+  )
+  (wire (pts (xy 147.066 64.516) (xy 147.066 63.5))
+    (stroke (width 0) (type default) (color 0 0 0 0))
+  )
+  (wire (pts (xy 94.234 59.436) (xy 95.758 59.436))
+    (stroke (width 0) (type default) (color 0 0 0 0))
+  )
+  (wire (pts (xy 94.234 62.992) (xy 94.234 64.516))
+    (stroke (width 0) (type default) (color 0 0 0 0))
+  )
+  (wire (pts (xy 116.078 64.516) (xy 123.698 64.516))
+    (stroke (width 0) (type default) (color 0 0 0 0))
+  )
+  (wire (pts (xy 140.462 45.974) (xy 145.034 45.974))
+    (stroke (width 0) (type default) (color 0 0 0 0))
+  )
+  (wire (pts (xy 147.066 63.5) (xy 149.098 63.5))
+    (stroke (width 0) (type default) (color 0 0 0 0))
+  )
+  (wire (pts (xy 74.168 60.452) (xy 81.026 60.452))
+    (stroke (width 0) (type default) (color 0 0 0 0))
+  )
+  (wire (pts (xy 147.32 60.96) (xy 147.32 59.436))
+    (stroke (width 0) (type default) (color 0 0 0 0))
+  )
+  (wire (pts (xy 94.234 59.436) (xy 94.234 60.452))
+    (stroke (width 0) (type default) (color 0 0 0 0))
+  )
+  (wire (pts (xy 149.098 60.96) (xy 147.32 60.96))
+    (stroke (width 0) (type default) (color 0 0 0 0))
+  )
+  (wire (pts (xy 81.788 62.992) (xy 94.234 62.992))
+    (stroke (width 0) (type default) (color 0 0 0 0))
+  )
+  (wire (pts (xy 118.618 59.436) (xy 118.618 45.974))
+    (stroke (width 0) (type default) (color 0 0 0 0))
+  )
+  (wire (pts (xy 123.698 64.516) (xy 147.066 64.516))
+    (stroke (width 0) (type default) (color 0 0 0 0))
+  )
+  (wire (pts (xy 94.234 64.516) (xy 95.758 64.516))
+    (stroke (width 0) (type default) (color 0 0 0 0))
+  )
+  (wire (pts (xy 116.078 59.436) (xy 118.618 59.436))
+    (stroke (width 0) (type default) (color 0 0 0 0))
+  )
+  (wire (pts (xy 118.618 45.974) (xy 120.396 45.974))
+    (stroke (width 0) (type default) (color 0 0 0 0))
+  )
+  (wire (pts (xy 123.698 64.516) (xy 123.698 67.818))
+    (stroke (width 0) (type default) (color 0 0 0 0))
+  )
+  (wire (pts (xy 147.32 59.436) (xy 118.618 59.436))
+    (stroke (width 0) (type default) (color 0 0 0 0))
+  )
+  (wire (pts (xy 74.168 62.992) (xy 81.788 62.992))
+    (stroke (width 0) (type default) (color 0 0 0 0))
+  )
+  (symbol (lib_id "power:GND") (at 123.698 67.818 0) (unit 1)
+    (in_bom yes) (on_board yes) (fields_autoplaced)
+    (property "Reference" "#PWR0102" (id 0) (at 123.698 74.168 0)
+      (effects (font (size 1.27 1.27)) hide)
+    )
+    (property "Value" "GND" (id 1) (at 123.698 72.39 0))
+    (property "Footprint" "" (id 2) (at 123.698 67.818 0)
+      (effects (font (size 1.27 1.27)) hide)
+    )
+    (property "Datasheet" "" (id 3) (at 123.698 67.818 0)
+      (effects (font (size 1.27 1.27)) hide)
+    )
+    (pin "1")
+  )
+  (symbol (lib_id "Connector_Generic:Conn_01x02") (at 69.088 62.992 180) (unit 1)
+    (in_bom yes) (on_board yes)
+    (property "Reference" "J1" (id 0) (at 70.104 57.404 0)
+      (effects (font (size 1.27 1.27)) (justify left))
+    )
+    (property "Value" "230VAC" (id 1) (at 71.628 66.802 0)
+      (effects (font (size 1.27 1.27)) (justify left))
+    )
+    (property "Footprint" "" (id 2) (at 69.088 62.992 0)
+      (effects (font (size 1.27 1.27)) hide)
+    )
+    (property "Datasheet" "~" (id 3) (at 69.088 62.992 0)
+      (effects (font (size 1.27 1.27)) hide)
+    )
+    (pin "1")
+    (pin "2")
+  )
+  (symbol (lib_id "Connector_Generic:Conn_01x02") (at 154.178 60.96 0) (unit 1)
+    (in_bom yes) (on_board yes)
+    (property "Reference" "J2" (id 0) (at 153.67 58.166 0)
+      (effects (font (size 1.27 1.27)) (justify left))
+    )
+    (property "Value" "5V+ Output" (id 1) (at 154.432 67.056 0)
+      (effects (font (size 1.27 1.27)) (justify left))
+    )
+    (property "Footprint" "" (id 2) (at 154.178 60.96 0)
+      (effects (font (size 1.27 1.27)) hide)
+    )
+    (property "Datasheet" "~" (id 3) (at 154.178 60.96 0)
+      (effects (font (size 1.27 1.27)) hide)
+    )
+    (pin "1")
+    (pin "2")
+  )
+  (symbol (lib_id "power:PWR_FLAG") (at 81.788 62.992 180) (unit 1)
+    (in_bom yes) (on_board yes)
+    (property "Reference" "#FLG0102" (id 0) (at 81.788 64.897 0)
+      (effects (font (size 1.27 1.27)) hide)
+    )
+    (property "Value" "PWR_FLAG" (id 1) (at 82.804 64.008 0)
+      (effects (font (size 0.5 0.5)) (justify right))
+    )
+    (property "Footprint" "" (id 2) (at 81.788 62.992 0)
+      (effects (font (size 1.27 1.27)) hide)
+    )
+    (property "Datasheet" "~" (id 3) (at 81.788 62.992 0)
+      (effects (font (size 1.27 1.27)) hide)
+    )
+    (pin "1")
+  )
+  (symbol (lib_id "power:PWR_FLAG") (at 81.026 60.452 0) (unit 1)
+    (in_bom yes) (on_board yes)
+    (property "Reference" "#FLG0101" (id 0) (at 81.026 58.547 0)
+      (effects (font (size 1.27 1.27)) hide)
+    )
+    (property "Value" "PWR_FLAG" (id 1) (at 83.566 59.436 0)
+      (effects (font (size 0.5 0.5)))
+    )
+    (property "Footprint" "" (id 2) (at 81.026 60.452 0)
+      (effects (font (size 1.27 1.27)) hide)
+    )
+    (property "Datasheet" "~" (id 3) (at 81.026 60.452 0)
+      (effects (font (size 1.27 1.27)) hide)
+    )
+    (pin "1")
+  )
+  (symbol (lib_id "Device:R") (at 136.652 45.974 90) (unit 1)
+    (in_bom yes) (on_board yes)
+    (property "Reference" "R1" (id 0) (at 136.652 43.434 90))
+    (property "Value" "2K" (id 1) (at 138.684 49.276 90))
+    (property "Footprint" "" (id 2) (at 136.652 47.752 90)
+      (effects (font (size 1.27 1.27)) hide)
+    )
+    (property "Datasheet" "~" (id 3) (at 136.652 45.974 0)
+      (effects (font (size 1.27 1.27)) hide)
+    )
+    (pin "1")
+    (pin "2")
+  )
+  (symbol (lib_id "Device:LED") (at 124.206 45.974 180) (unit 1)
+    (in_bom yes) (on_board yes)
+    (property "Reference" "D1" (id 0) (at 125.222 42.164 0))
+    (property "Value" "PWR LED" (id 1) (at 128.016 49.022 0))
+    (property "Footprint" "" (id 2) (at 124.206 45.974 0)
+      (effects (font (size 1.27 1.27)) hide)
+    )
+    (property "Datasheet" "~" (id 3) (at 124.206 45.974 0)
+      (effects (font (size 1.27 1.27)) hide)
+    )
+    (pin "1")
+    (pin "2")
+  )
+  (symbol (lib_id "power:GND") (at 145.034 48.768 0) (unit 1)
+    (in_bom yes) (on_board yes) (fields_autoplaced)
+    (property "Reference" "#PWR0101" (id 0) (at 145.034 55.118 0)
+      (effects (font (size 1.27 1.27)) hide)
+    )
+    (property "Value" "GND" (id 1) (at 145.034 53.34 0))
+    (property "Footprint" "" (id 2) (at 145.034 48.768 0)
+      (effects (font (size 1.27 1.27)) hide)
+    )
+    (property "Datasheet" "" (id 3) (at 145.034 48.768 0)
+      (effects (font (size 1.27 1.27)) hide)
+    )
+    (pin "1")
+  )
+  (symbol (lib_id "Converter_ACDC:IRM-03-5") (at 105.918 61.976 0) (unit 1)
+    (in_bom yes) (on_board yes)
+    (property "Reference" "PS1" (id 0) (at 105.918 55.372 0))
+    (property "Value" "IRM-03-5" (id 1) (at 106.68 68.58 0))
+    (property "Footprint" "Converter_ACDC:Converter_ACDC_MeanWell_IRM-03-xx_THT" (id 2) (at 105.918 70.866 0)
+      (effects (font (size 1.27 1.27)) hide)
+    )
+    (property "Datasheet" "https://www.meanwell.com/Upload/PDF/IRM-03/IRM-03-SPEC.PDF" (id 3) (at 105.918 72.136 0)
+      (effects (font (size 1.27 1.27)) hide)
+    )
+    (pin "1")
+    (pin "14")
+    (pin "16")
+    (pin "3")
+    (pin "5")
   )
   (sheet_instances
     (path "/" (page "1"))
   )
+  (symbol_instances
+    (path "/64281808-2d8f-46cb-a0cf-39a334bcf5a1"
+      (reference "#FLG0101") (unit 1) (value "PWR_FLAG") (footprint "")
+    )
+    (path "/5b5137b4-6f7e-4988-86c9-c80b56c27e76"
+      (reference "#FLG0102") (unit 1) (value "PWR_FLAG") (footprint "")
+    )
+    (path "/f232a31d-55ae-45e1-aca8-905e73c4eddc"
+      (reference "#PWR0101") (unit 1) (value "GND") (footprint "")
+    )
+    (path "/27d09938-6d3d-4a4b-84db-4f57b6dac4d7"
+      (reference "#PWR0102") (unit 1) (value "GND") (footprint "")
+    )
+    (path "/ee96581b-d583-46b9-83f7-9d8f6920a4da"
+      (reference "D1") (unit 1) (value "PWR LED") (footprint "")
+    )
+    (path "/3cccc916-9468-40cf-9875-cd5cd535ee1b"
+      (reference "J1") (unit 1) (value "230VAC") (footprint "")
+    )
+    (path "/467062e1-4244-4afe-a712-ae965d0f31b7"
+      (reference "J2") (unit 1) (value "5V+ Output") (footprint "")
+    )
+    (path "/f847cecc-f311-46bd-b1ed-a46a90ce9cc0"
+      (reference "PS1") (unit 1) (value "IRM-03-5") (footprint "Converter_ACDC:Converter_ACDC_MeanWell_IRM-03-xx_THT")
+    )
+    (path "/c4c23962-2dc3-463f-a8a3-012aec07cf9f"
+      (reference "R1") (unit 1) (value "2K") (footprint "")
+    )
+  )
 )

Commit message: adding component placing adding routing adding final touches
Parts:
- removed J1: 230VAC, symbol Connector_Generic:Conn_01x02
- removed PS1: IRM-03-5, Converter_ACDC:Converter_ACDC_MeanWell_IRM-03-xx_THT, symbol Converter_ACDC:IRM-03-5
- added H1, H2, H3, H4: MountingHole, MountingHole:MountingHole_3.2mm_M3_ISO7380, symbol Mechanical:MountingHole
- added J1: 230VAC, Phoenix_Contact_1711026:SHDR2W110P0X500_1X2_1000X1120X, symbol 1711026:1711026
- added PS1: IRM-03-5, MeanWell_IRM-03-5:IRM0312, symbol IRM-03-5:IRM-03-5
- D1: footprint (none) -> LED_THT:LED_D5.0mm
- J2: footprint (none) -> Connector_JST:JST_XH_B2B-XH-A_1x02_P2.50mm_Vertical
- R1: footprint (none) -> Resistor_THT:R_Axial_DIN0207_L6.3mm_D2.5mm_P7.62mm_Horizontal
Connections:
- net GND: now also J2.1 (Pin_1), PS1.4 (-V); no longer J2.2 (Pin_2)
- net +5V: now reaches D1.2 (A)
- net +5V: now also J2.2 (Pin_2), PS1.5 (+V); no longer J2.1 (Pin_1)
- new net Line: J1.2, PS1.1 (AC/L)
- new net Neutral: J1.1, PS1.2 (AC/N)
Other:
- note added: "Mounting Holes"
- moved on the sheet: D1, J2, R1
